File: UDB.kicad_pcb (KiCad board)
At the start: 4 copper layers, 18 x 16.5 mm, 14 parts, among them J1 TYPE-C-31-M12_13, J2 SM04B-SRSS-TB(LF)(SN), U1 TPD4E05U06DQAR

Commit message: added kikit panel assembly
Parts:
- removed G1: Unified-Daughterboard-Logo, Unified-Daughterboard-Logo:Unified-Daughterboard-Logo.pretty
Changed lines of the file:
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@@
       ))
-  )
-  (footprint "Unified-Daughterboard-Logo:Unified-Daughterboard-Logo.pretty" (layer "B.Cu")
-    (at 75.0025 67.143 180)
-    (property "Sheetfile" "File: UDB.kicad_sch")
-    (property "Sheetname" "")
-    (property "exclude_from_bom" "")
-    (attr through_hole exclude_from_pos_files exclude_from_bom)
-    (fp_text reference "G1" (at 0 0) (layer "B.SilkS") hide
-      (effects (font (size 1.524 1.524) (thickness 0.3)) (justify mirror))
-    )
-    (fp_text value "Unified-Daughterboard-Logo" (at 0.75 0) (layer "B.SilkS") hide
-      (effects (font (size 1.524 1.524) (thickness 0.3)) (justify mirror))
-    )
-    (fp_poly (pts
-        (xy -1.984345 3.315323)
-        (xy -0.995318 3.315284)
-        (xy -1.795436 2.733919)
-        (xy -1.489845 1.793287)
-        (xy -2.290007 2.374593)
-        (xy -3.090169 1.793287)
-        (xy -2.784578 2.73392)
-        (xy -3.584696 3.315285)
-        (xy -2.595669 3.315323)
-        (xy -2.290007 4.255932)
-      ) (layer "B.SilkS") (width 0) (fill solid))
-    (fp_poly (pts
-        (xy 4.010971 -1.04053)
-        (xy 4.999998 -1.040569)
-        (xy 4.199881 -1.621933)
-        (xy 4.505472 -2.562566)
-        (xy 3.705309 -1.98126)
-        (xy 2.905147 -2.562566)
-        (xy 3.210739 -1.621933)
-        (xy 2.410621 -1.040567)
-        (xy 3.399648 -1.04053)
-        (xy 3.705309 -0.099921)
-      ) (layer "B.SilkS") (width 0) (fill solid))
-    (fp_poly (pts
-        (xy 2.59567 3.315322)
-        (xy 3.584697 3.315284)
-        (xy 2.784579 2.733919)
-        (xy 3.090169 1.793287)
-        (xy 2.290008 2.374592)
-        (xy 1.489846 1.793287)
-        (xy 1.795436 2.733919)
-        (xy 0.995319 3.315285)
-        (xy 1.984346 3.315323)
-        (xy 2.290008 4.255932)
-      ) (layer "B.SilkS") (width 0) (fill solid))
-    (fp_poly (pts
-        (xy -3.399648 1.367326)
-        (xy -2.41062 1.367288)
-        (xy -3.210738 0.785923)
-        (xy -2.905148 -0.15471)
-        (xy -3.705309 0.426596)
-        (xy -4.505471 -0.15471)
-        (xy -4.199881 0.785923)
-        (xy -4.999999 1.367289)
-        (xy -4.010971 1.367326)
-        (xy -3.705309 2.307936)
-      ) (layer "B.SilkS") (width 0) (fill solid))
-    (fp_poly (pts
-        (xy 2.59567 -2.988526)
-        (xy 3.584697 -2.988565)
-        (xy 2.784579 -3.569929)
-        (xy 3.090169 -4.510561)
-        (xy 2.290008 -3.929257)
-        (xy 1.489846 -4.510561)
-        (xy 1.795436 -3.569929)
-        (xy 0.995319 -2.988563)
-        (xy 1.984346 -2.988526)
-        (xy 2.290008 -2.047917)
-      ) (layer "B.SilkS") (width 0) (fill solid))
-    (fp_poly (pts
-        (xy 0.305662 -3.732595)
-        (xy 1.29469 -3.732633)
-        (xy 0.494571 -4.313998)
-        (xy 0.800162 -5.25463)
-        (xy 0 -4.673325)
-        (xy -0.800162 -5.25463)
-        (xy -0.494571 -4.313998)
-        (xy -1.294689 -3.732632)
-        (xy -0.305662 -3.732595)
-        (xy 0 -2.791985)
-      ) (layer "B.SilkS") (width 0) (fill solid))
-    (fp_poly (pts
-        (xy -1.984346 -2.988526)
-        (xy -0.995318 -2.988565)
-        (xy -1.795436 -3.569929)
-        (xy -1.489845 -4.510561)
-        (xy -2.290007 -3.929257)
-        (xy -3.090169 -4.510561)
-        (xy -2.784579 -3.569929)
-        (xy -3.584696 -2.988563)
-        (xy -2.595669 -2.988526)
-        (xy -2.290007 -2.047917)
-      ) (layer "B.SilkS") (width 0) (fill solid))
-    (fp_poly (pts
-        (xy 4.010971 1.317119)
-        (xy 4.999998 1.31708)
-        (xy 4.199881 0.735716)
-        (xy 4.505472 -0.204917)
-        (xy 3.705309 0.376388)
-        (xy 2.905147 -0.204917)
-        (xy 3.210739 0.735716)
-        (xy 2.410621 1.317081)
-        (xy 3.399648 1.317119)
-        (xy 3.705309 2.257728)
-      ) (layer "B.SilkS") (width 0) (fill solid))
-    (fp_poly (pts
-        (xy -3.399648 -1.04053)
-        (xy -2.41062 -1.040569)
-        (xy -3.210738 -1.621933)
-        (xy -2.905148 -2.562566)
-        (xy -3.70531 -1.98126)
-        (xy -4.505471 -2.562566)
-        (xy -4.199881 -1.621933)
-        (xy -4.999999 -1.040567)
-        (xy -4.010971 -1.04053)
-        (xy -3.70531 -0.099921)
-      ) (layer "B.SilkS") (width 0) (fill solid))
-    (fp_poly (pts
-        (xy 0.305662 4.059391)
-        (xy 1.29469 4.059353)
-        (xy 0.494571 3.477988)
-        (xy 0.800162 2.537355)
-        (xy 0 3.118661)
-        (xy -0.800162 2.537355)
-        (xy -0.494571 3.477988)
-        (xy -1.294689 4.059354)
-        (xy -0.305662 4.059391)
-        (xy 0 5)
-      ) (layer "B.SilkS") (width 0) (fill solid))
   )
   (gr_arc (start 82.0045 56.543) (mid 83.418714 57.128786) (end 84.0045 58.543) (layer "Edge.Cuts") (width 0.15))
