File: UDB.kicad_sch (KiCad schematic)
At the start: 14 parts, among them J1 TYPE-C-31-M12_13, J2 X1224WRS-04-LPV01, U1 TPD4E05U06DQAR

Commit message: added kikit panel assembly
Parts:
- D1: LCSC (none) -> C708002; LCSC Part Number C708002 -> (none)
- F1: LCSC (none) -> C135342; LCSC Part Number C135342 -> (none)
- J1: JLCPCB_CORRECTION (none) -> 0; 3; 0; LCSC (none) -> C165948; LCSC Part Number C165948 -> (none)
- J2: JLCPCB_CORRECTION (none) -> 0; 2; 0; LCSC (none) -> C528030; LCSC Part Number C528030 -> (none)
- L1: LCSC (none) -> C33600; LCSC Part Number C33600 -> (none)
- R1: LCSC (none) -> C138073; LCSC Part Number C25905 -> (none); Manufacturer Uniroyal -> (none); Manufacturer Part Number 0402WGF5101TCE -> (none)
- R2: LCSC (none) -> C138073
- U1: JLCPCB_CORRECTION (none) -> 0; 0; 270; LCSC (none) -> C138714; LCSC Part Number C138714 -> (none)
Changed lines of the file:
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@@
       (effects (font (size 1.27 1.27)) hide)
     )
-    (property "LCSC Part Number" "C528030" (id 7) (at 241.3 77.47 0)
+    (property "LCSC" "C528030" (id 7) (at 241.3 77.47 0)
+      (effects (font (size 1.27 1.27)) hide)
+    )
+    (property "JLCPCB_CORRECTION" "0; 2; 0" (id 8) (at 241.3 77.47 0)
       (effects (font (size 1.27 1.27)) hide)
     )
@@
       (effects (font (size 1.27 1.27)) hide)
     )
-    (property "Manufacturer" "Uniroyal" (id 5) (at 59.055 42.545 90)
-      (effects (font (size 1.27 1.27)) hide)
-    )
-    (property "Manufacturer Part Number" "0402WGF5101TCE" (id 6) (at 59.055 42.545 90)
-      (effects (font (size 1.27 1.27)) hide)
-    )
-    (property "LCSC Part Number" "C25905" (id 7) (at 59.055 42.545 90)
+    (property "Manufacturer" "" (id 5) (at 59.055 42.545 90)
+      (effects (font (size 1.27 1.27)) hide)
+    )
+    (property "Manufacturer Part Number" "" (id 6) (at 59.055 42.545 90)
+      (effects (font (size 1.27 1.27)) hide)
+    )
+    (property "LCSC" "C138073" (id 7) (at 59.055 42.545 90)
       (effects (font (size 1.27 1.27)) hide)
     )
@@
       (effects (font (size 1.27 1.27)) hide)
     )
+    (property "LCSC" "C138073" (id 5) (at 59.055 47.625 0)
+      (effects (font (size 1.27 1.27)) hide)
+    )
+    (property "Manufacturer" "" (id 6) (at 59.055 47.625 0)
+      (effects (font (size 1.27 1.27)) hide)
+    )
+    (property "Manufacturer Part Number" "" (id 7) (at 59.055 47.625 0)
+      (effects (font (size 1.27 1.27)) hide)
+    )
     (pin "1")
     (pin "2")
@@
       (effects (font (size 1.27 1.27)) hide)
     )
-    (property "LCSC Part Number" "C708002" (id 7) (at 113.665 90.17 0)
+    (property "LCSC" "C708002" (id 7) (at 113.665 90.17 0)
       (effects (font (size 1.27 1.27)) hide)
     )
@@
       (effects (font (size 1.27 1.27)) hide)
     )
-    (property "LCSC Part Number" "C165948" (id 7) (at 40.005 59.055 0)
+    (property "LCSC" "C165948" (id 7) (at 40.005 59.055 0)
+      (effects (font (size 1.27 1.27)) hide)
+    )
+    (property "JLCPCB_CORRECTION" "0; 3; 0" (id 8) (at 40.005 59.055 0)
       (effects (font (size 1.27 1.27)) hide)
     )
@@
       (effects (font (size 1.27 1.27)) hide)
     )
-    (property "LCSC Part Number" "C138714" (id 8) (at 111.125 43.815 0)
+    (property "LCSC" "C138714" (id 8) (at 111.125 43.815 0)
+      (effects (font (size 1.27 1.27)) hide)
+    )
+    (property "JLCPCB_CORRECTION" "0; 0; 270" (id 9) (at 111.125 43.815 0)
       (effects (font (size 1.27 1.27)) hide)
     )
@@
       (effects (font (size 1.27 1.27)) hide)
     )
-    (property "LCSC Part Number" "C135342" (id 6) (at 107.315 85.09 90)
+    (property "LCSC" "C135342" (id 6) (at 107.315 85.09 90)
       (effects (font (size 1.27 1.27)) hide)
     )
@@
       (effects (font (size 1.27 1.27)) hide)
     )
-    (property "LCSC Part Number" "C33600" (id 8) (at 32.385 114.935 0)
-      (effects (font (size 1.27 1.27)) hide)
-    )
+    (property "LCSC" "C33600" (id 8) (at 32.385 114.935 0)
+      (effects (font (size 1.27 1.27)) hide)
+    )
